Commit message: adding difflink collisions

File: unity-sim/Assets/RoverDescription/rover.urdf (robot description, URDF)
Before this commit: robot Banksia, 62 links, 65 joints
Links:
- link left_difflink: geometry collision mesh filename=file://Assets/RoverDescription/banksia/meshes/left_difflink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; visual mesh filename=file://Assets/RoverDescription/banksia/meshes/left_difflink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
- link right_difflink: geometry collision mesh filename=file://Assets/RoverDescription/banksia/meshes/right_difflin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; visual mesh filename=file://Assets/RoverDescription/banksia/meshes/right_difflin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
