Commit message: Added missing realsense TF frames; fixed CAN thread not exiting when play is exited.

File: unity-sim/Assets/RoverDescription/banksia.urdf (robot description, URDF)
Before this commit: robot Banksia, 31 links, 30 joints
Links:
- added link d415_color_frame
- added link d415_color_optical_frame
- added link d415_depth_frame
- added link d415_depth_optical_frame
- added link d415_infra1_frame
- added link d415_infra1_optical_frame
- added link d415_infra2_frame
- added link d415_infra2_optical_frame
- link bl_ankle: geometry collision box size=0.012 0.03 0.06; collision box size=0.012 0.076 0.06
- link bl_wheel: geometry collision cylinder length=0.16 radius=0.157; visual mesh filename=file://Assets/RoverDescription/banksia/meshes/bl_wheel.stl
- link br_ankle: geometry collision box size=0.012 0.03 0.06; collision box size=0.012 0.076 0.06
- link br_wheel: geometry collision cylinder length=0.16 radius=0.157; visual mesh filename=file://Assets/RoverDescription/banksia/meshes/br_wheel.stl
- link chassis: geometry collision box size=0.48 0.545 0.175; visual mesh filename=file://Assets/RoverDescription/banksia/meshes/chassis.stl
- link clam: geometry collision box size=0.02 0.25 0.04; collision box size=0.02 0.25 0.04
- link d415_link: geometry collision box size=0.02005 0.099 0.023; visual mesh filename=file://Assets/RoverDescription/realsense2/meshes/d415.stl
- link diffbar: geometry collision cylinder length=0.41 radius=0.01; collision cylinder length=0.41 radius=0.01
- link fl_ankle: geometry collision box size=0.012 0.03 0.06; collision box size=0.012 0.076 0.06
- link fl_wheel: geometry collision cylinder length=0.16 radius=0.157; visual mesh filename=file://Assets/RoverDescription/banksia/meshes/fl_wheel.stl
- link fr_ankle: geometry collision box size=0.012 0.03 0.06; collision box size=0.012 0.076 0.06
- link fr_wheel: geometry collision cylinder length=0.16 radius=0.157; visual mesh filename=file://Assets/RoverDescription/banksia/meshes/fr_wheel.stl
- link left_difflink: geometry visual mesh filename=file://Assets/RoverDescription/banksia/meshes/left_difflink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
- link left_leg: geometry collision box size=0.106 0.065 0.077; collision box size=0.107 0.065 0.077
- link livox_frame: geometry visual mesh filename=file://Assets/RoverDescription/auto_mount/meshes/mid-360-as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
- link mount: geometry visual mesh filename=file://Assets/RoverDescription/auto_mount/meshes/mount.stl scale=1 1 1
- link right_difflink: geometry visual mesh filename=file://Assets/RoverDescription/banksia/meshes/right_difflin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
- link right_leg: geometry collision box size=0.106 0.065 0.077; collision box size=0.107 0.065 0.077
Joints:
- added joint d415_color_joint: type fixed, parent d415_link, child d415_color_frame, origin xyz=0 0.015 0 rpy=0 0 0
- added joint d415_color_optical_joint: type fixed, parent d415_color_frame, child d415_color_optical_frame, origin xyz=0 0 0 rpy=-1.5707963267948966 0 -1.5707963267948966
- added joint d415_depth_joint: type fixed, parent d415_link, child d415_depth_frame, origin xyz=0 0 0 rpy=0 0 0
- added joint d415_depth_optical_joint: type fixed, parent d415_depth_frame, child d415_depth_optical_frame, origin xyz=0 0 0 rpy=-1.5707963267948966 0 -1.5707963267948966
- added joint d415_infra1_joint: type fixed, parent d415_link, child d415_infra1_frame, origin xyz=0 0.0 0 rpy=0 0 0
- added joint d415_infra1_optical_joint: type fixed, parent d415_infra1_frame, child d415_infra1_optical_frame, origin xyz=0 0 0 rpy=-1.5707963267948966 0 -1.5707963267948966
- added joint d415_infra2_joint: type fixed, parent d415_link, child d415_infra2_frame, origin xyz=0 -0.055 0 rpy=0 0 0
- added joint d415_infra2_optical_joint: type fixed, parent d415_infra2_frame, child d415_infra2_optical_frame, origin xyz=0 0 0 rpy=-1.5707963267948966 0 -1.5707963267948966
