Commit message: Updating Banksia Auto to work with the new mount, and removing the tmux from shell aliases

File: unity-sim/Assets/RoverDescription/auto_mount/urdf/livox.xacro (robot description, xacro)
@@ -1,47 +1,75 @@
 <?xml version="1.0" encoding="utf-8" ?>
 <robot xmlns:xacro="http://www.ros.org/wiki/xacro">
-  <link name="livox_frame">
-    <visual>
-        <origin xyz="0 0.0055 0" rpy="0 0 3.14159" />
-        <geometry>
-            <mesh filename="file://$(find rover_description)/auto_mount/meshes/mid-360-asm.stl"/>
-        </geometry>
-    </visual>
-  </link>
-  <gazebo reference="livox_frame">
-        <sensor name="gpu_lidar" type="gpu_lidar">
-            <update_rate>10</update_rate>
-            <topic>livox/lidar</topic>
-            <gz_frame_id>livox_frame</gz_frame_id>
-            <update_rate>10</update_rate>
-            <ray>
-              <scan>
-                <horizontal>
-                  <samples>720</samples>      <!-- MID-360 0.5° resolution -->
-                  <resolution>1</resolution>
-                  <!-- MID-360 HFOV = 360° -->
-                  <min_angle>-3.14156</min_angle>
-                  <max_angle>3.14156</max_angle>
-                </horizontal>
-                <vertical>
-                  <samples
-                        >40</samples>       <!-- MID-360 point cloud density -->
-                  <resolution>1</resolution>
-                  <!-- MID-360 VFOV = 59° -->
-                  <min_angle>0</min_angle>
-                  <max_angle>0.9774</max_angle>
-                </vertical>
-              </scan>
-              <range>
-                <min
-                    >0.01</min>                 <!-- MID-360 min. detection range -->
-                <max
-                    >40.0</max>                 <!-- MID-360 max. detection range -->
-                <resolution>0.01</resolution>
-              </range>
-            </ray>
-            <always_on>1</always_on>
-            <visualize>true</visualize>
-        </sensor>
-  </gazebo>
+    <xacro:macro name="sensor_livox" params="parent *origin">
+        <link name="livox_frame">
+            <visual>
+                <origin xyz="0 0.0055 0" rpy="0 0 3.14159" />
+                <geometry>
+                    <mesh filename="file://$(arg rover_description_dir)/auto_mount/meshes/mid-360-asm.stl"/>
+                </geometry>
+                <visibility_flags>0x02</visibility_flags> <!-- Bit 1 -->
+            </visual>
+        </link>
+        <joint name="livox_joint" type="fixed">
+            <xacro:insert_block name="origin" />
+            <parent link="${parent}" />
+            <child link="livox_frame" />
+        </joint>
+    </xacro:macro>
+    <!-- Gazebo sensor plugin for the Livox MID-360 LiDAR (does not affect IRL) -->
+    <xacro:if value="$(arg gazebo)">
+        <gazebo reference="livox_frame">
+            <visibility_flags>0x02</visibility_flags>
+            <sensor name="mid360" type="gpu_lidar">
+                <update_rate>20</update_rate>
+                <topic>livox/lidar</topic>
+                <gz_frame_id>livox_frame</gz_frame_id>
+                <visibility_mask>0xFFFFFFFD</visibility_mask> <!-- All bits except bit 1 -->
+                <ray>
+                    <scan>
+                        <horizontal>
+                            <samples>500</samples>      <!-- MID-360 0.5° resolution -->
+                            <resolution>1.0</resolution>
+                            <!-- MID-360 HFOV = 360° -->
+                            <min_angle>-3.14156</min_angle>
+                            <max_angle>3.14156</max_angle>
+                        </horizontal>
+                        <vertical>
+                            <samples>40</samples>       <!-- MID-360 point cloud density -->
+                            <resolution>1.0</resolution>
+                            <!-- MID-360 VFOV = 59° -->
+                            <min_angle>-0.122173</min_angle>
+                            <max_angle>0.907571</max_angle>
+                        </vertical>
+                    </scan>
+                    <range>
+                        <min>0.05</min>                 <!-- MID-360 min. detection range -->
+                        <max>40.0</max>                 <!-- MID-360 max. detection range -->
+                        <resolution>0.01</resolution>
+                    </range>
+                </ray>
+                <always_on>1</always_on>
+                <visualize>false</visualize>
+            </sensor>
+            <sensor name="mid360_imu" type="imu">
+                <update_rate>200</update_rate>
+                <topic>livox/imu</topic>
+                <gz_frame_id>livox_frame</gz_frame_id>
+                <always_on>1</always_on>
+                <visualize>false</visualize>
+                <imu>
+                    <angular_velocity>
+                        <x><noise type="gaussian"><mean>0.0</mean><stddev>2e-4</stddev></noise></x>
+                        <y><noise type="gaussian"><mean>0.0</mean><stddev>2e-4</stddev></noise></y>
+                        <z><noise type="gaussian"><mean>0.0</mean><stddev>2e-4</stddev></noise></z>
+                    </angular_velocity>
+                    <linear_acceleration>
+                        <x><noise type="gaussian"><mean>0.0</mean><stddev>1.7e-2</stddev></noise></x>
+                        <y><noise type="gaussian"><mean>0.0</mean><stddev>1.7e-2</stddev></noise></y>
+                        <z><noise type="gaussian"><mean>0.0</mean><stddev>1.7e-2</stddev></noise></z>
+                    </linear_acceleration>
+                </imu>
+            </sensor>
+        </gazebo>
+    </xacro:if>
 </robot>

File: unity-sim/Assets/RoverDescription/banksia.urdf (robot description, URDF)
Before this commit: robot Banksia, 31 links, 30 joints
Links:
- link bl_ankle: geometry collision box size=0.012 0.03 0.06; collision box size=0.012 0.076 0.06
- link bl_wheel: geometry collision cylinder length=0.16 radius=0.157; visual mesh filename=file:///nix/store/5f92nb8rag9mzzwjmxkam8xvzanz6ncm-ros-jazz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
- link br_ankle: geometry collision box size=0.012 0.03 0.06; collision box size=0.012 0.076 0.06
- link br_wheel: geometry collision cylinder length=0.16 radius=0.157; visual mesh filename=file:///nix/store/5f92nb8rag9mzzwjmxkam8xvzanz6ncm-ros-jazz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
- link chassis: geometry collision box size=0.48 0.545 0.175; visual mesh filename=file:///nix/store/5f92nb8rag9mzzwjmxkam8xvzanz6ncm-ros-jazz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
- link clam: geometry collision box size=0.02 0.25 0.04; collision box size=0.02 0.25 0.04
- link d415_link: geometry collision box size=0.02005 0.099 0.023; visual mesh filename=file:///nix/store/5f92nb8rag9mzzwjmxkam8xvzanz6ncm-ros-jazz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
- link diffbar: geometry collision cylinder length=0.41 radius=0.01; collision cylinder length=0.41 radius=0.01
- link fl_ankle: geometry collision box size=0.012 0.03 0.06; collision box size=0.012 0.076 0.06
- link fl_wheel: geometry collision cylinder length=0.16 radius=0.157; visual mesh filename=file:///nix/store/5f92nb8rag9mzzwjmxkam8xvzanz6ncm-ros-jazz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
- link fr_ankle: geometry collision box size=0.012 0.03 0.06; collision box size=0.012 0.076 0.06
- link fr_wheel: geometry collision cylinder length=0.16 radius=0.157; visual mesh filename=file:///nix/store/5f92nb8rag9mzzwjmxkam8xvzanz6ncm-ros-jazz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
- link left_difflink: geometry visual mesh filename=file:///nix/store/5f92nb8rag9mzzwjmxkam8xvzanz6ncm-ros-jazz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
- link left_leg: geometry collision box size=0.106 0.065 0.077; collision box size=0.107 0.065 0.077
- link livox_frame: geometry visual mesh filename=file:///nix/store/5f92nb8rag9mzzwjmxkam8xvzanz6ncm-ros-jazz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
- link mount: geometry visual mesh filename=file:///nix/store/5f92nb8rag9mzzwjmxkam8xvzanz6ncm-ros-jazz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 scale=1 1 1
- link right_difflink: geometry visual mesh filename=file:///nix/store/5f92nb8rag9mzzwjmxkam8xvzanz6ncm-ros-jazz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
- link right_leg: geometry collision box size=0.106 0.065 0.077; collision box size=0.107 0.065 0.077
